File: Hardware/PowerConverter.kicad_pcb (KiCad board)
At the start: 2 copper layers, 55.9 x 33 mm, 12 parts, among them J1 Barrel_Jack, J2 Screw_Terminal_01x04, J3 Screw_Terminal_01x04, U1 LM317_3PinPackage, U2 LM317_3PinPackage

Commit message: Initial release for V1
Parts:
- added G***: LOGO, Hardware:EE-EmergeLogo, B.Cu at (144.8, 113.0)
- moved C1 29.2 mm to (134.6, 97.5)
- moved C2 29.2 mm to (134.6, 115.2)
- moved D1 29.2 mm to (125.3, 97.2)
- moved J1 29.2 mm to (127.6, 104.8)
- moved J2 29.2 mm to (166.6, 115.7)
- moved J3 29.2 mm to (166.6, 99.2)
- moved R1 29.2 mm to (134.6, 110.5)
- moved R2 29.2 mm to (134.6, 108.0)
- moved R3 29.2 mm to (134.6, 92.7)
- moved R4 29.2 mm to (134.6, 90.2)
- moved U1 29.2 mm to (148.6, 110.5)
- moved U2 29.2 mm to (148.6, 94.0)
Other:
- board text added: "Designer: Sean Alling Rev: 1.0"
