File: Hardware/PowerConverter.sch (KiCad schematic (older format))
At the start: 12 parts, among them J1 Barrel_Jack, J2 Screw_Terminal_01x04, J3 Screw_Terminal_01x04, U1 LM317_3PinPackage, U2 LM317_3PinPackage

Commit message: Initial release for V1
Other:
- moved on the sheet: C1, C2, D1, J1, R1, R2, R3, R4, U1, U2
